File: payload/hardware/payload.kicad_sch (KiCad schematic)
At the start: 0 parts

Commit message: update name
Other:
- company: SaganSat -> Orbitalis
Changed lines of the file:
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@@
     (date "22/05/2023")
     (rev "1.0")
-    (company "SaganSat")
+    (company "Orbitalis")
     (comment 1 "Felipe Costa Juliano")
     (comment 2 "João Victor M. S. Dias")
